File: flipdot.kicad_pcb (KiCad board)
At the start: 2 copper layers, 45.7 x 33 mm, 54 parts, among them P2 FLIPDOT, P3 CAN, P4 VCC, P5 ESP8266-1, P6 CONN_02X03, P7 JTAG, SW1 SW_Push, SW2 SW_Push, U1 TJA1051T/3, U2 STM32F072C8Tx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

Commit message: add mounting holes
Parts:
- added REF**: 1pin, Connectors:1pin, F.Cu at (221.0, 52.1)
- added REF**: 1pin, Connectors:1pin, F.Cu at (192.4, 52.1)
- added REF**: 1pin, Connectors:1pin, F.Cu at (227.3, 78.1)
- moved SW1 1.50 mm to (197.5, 52.0)
- moved SW2 1.50 mm to (197.5, 56.0)
Routing:
- net BOOT: track 31.2 -> 29.7 mm
- net NRST: track 53.7 -> 52.2 mm
- added copper zone on F.Cu, net +3V3
Other:
- board text added: "flipdot control v0.1.2"
- board text removed: "flipdot control v0.1.1"
